Commit message: README.md update

File: ur_description/urdf/ur10e.xacro (robot description, xacro)
@@ -20,8 +20,9 @@
   <xacro:include filename="$(find realsense2_description)/urdf/test_d435i_camera.urdf.xacro" />
   <xacro:realsense2_camera parent="base_link" use_nominal_extrinsics="true">
-<!--      <origin xyz="0.758 -0.715 0.491 " rpy="3.067 2.351 -1.724"/>-->
-<!--    2.402 = -0.74 + pi &ndash;&gt; para fazer a calib, meter a garra (tool0_controller) e gravar tudo igual exceto esta rotacao-->
-<!--      <origin xyz="0.758 -0.715 0.491 " rpy="3.131 2.402 -1.711"/>-->
-      <origin xyz="0.7 -0.833 0.424 " rpy="3.073 2.627 -1.650"/>
+<!--    For this manual calibration, drag the gripper (tool0_controller) to the camera mass
+        center and record here the tf values (/base_link to /tool0_controller).-->
+<!--    The second rotation value (P) you should add pi constant: 2.627 = −0,515 + pi -->
+<!--      <origin xyz="0.7 -0.833 0.424 " rpy="3.073 2.627 -1.650"/>-->
+      <origin xyz="0.857 -0.075 0.378 " rpy="-3.075 3,330 -2.741"/>
   </xacro:realsense2_camera>
 <!--  <xacro:realsense2_camera use_nominal_extrinsics="true">-->

Commit message: README.md update

File: ur_description/urdf/ur10e.xacro (robot description, xacro)
@@ -23,6 +23,5 @@
         center and record here the tf values (/base_link to /tool0_controller).-->
 <!--    The second rotation value (P) you should add pi constant: 2.627 = −0,515 + pi -->
-<!--      <origin xyz="0.7 -0.833 0.424 " rpy="3.073 2.627 -1.650"/>-->
-      <origin xyz="0.857 -0.075 0.378 " rpy="-3.075 3,330 -2.741"/>
+      <origin xyz="0.7 -0.833 0.424 " rpy="3.073 2.627 -1.650"/>
   </xacro:realsense2_camera>
 <!--  <xacro:realsense2_camera use_nominal_extrinsics="true">-->

Commit message: Major advances: Created Gripper Controller Created Arm Controller Created 1st use case demo, using both new controllers

File: ur_description/urdf/ur10e.xacro (robot description, xacro)
@@ -23,5 +23,5 @@
         center and record here the tf values (/base_link to /tool0_controller).-->
 <!--    The second rotation value (P) you should add pi constant: 2.627 = −0,515 + pi -->
-      <origin xyz="0.7 -0.833 0.424 " rpy="3.073 2.627 -1.650"/>
+      <origin xyz="0.793 -0.804 0.425" rpy="-3.114 2.454 -1.582"/>
   </xacro:realsense2_camera>
 <!--  <xacro:realsense2_camera use_nominal_extrinsics="true">-->

Commit message: Creating an Utils Library for Arm and Gripper control (not working yet) Creating some tests scripts for testing particular actions for the demo1.py upgrade

File: ur_description/urdf/ur10e.xacro (robot description, xacro)
@@ -23,5 +23,6 @@
         center and record here the tf values (/base_link to /tool0_controller).-->
 <!--    The second rotation value (P) you should add pi constant: 2.627 = −0,515 + pi -->
-      <origin xyz="0.793 -0.804 0.425" rpy="-3.114 2.454 -1.582"/>
+<!--      <origin xyz="0.785 -0.839 0.426" rpy="-3.104 2.471 -1.613"/>-->
+      <origin xyz="0.800 -0.792 0.437" rpy="3.112 2.471 -1.558"/>
   </xacro:realsense2_camera>
 <!--  <xacro:realsense2_camera use_nominal_extrinsics="true">-->

Commit message: just for testing gripper force value

File: ur_description/urdf/ur10e.xacro (robot description, xacro)
@@ -24,5 +24,5 @@
 <!--    The second rotation value (P) you should add pi constant: 2.627 = −0,515 + pi -->
 <!--      <origin xyz="0.785 -0.839 0.426" rpy="-3.104 2.471 -1.613"/>-->
-      <origin xyz="0.800 -0.792 0.437" rpy="3.112 2.471 -1.558"/>
+      <origin xyz="0.797 -0.803 0.432" rpy="3.135 2.462 -1.577"/>
   </xacro:realsense2_camera>
 <!--  <xacro:realsense2_camera use_nominal_extrinsics="true">-->
