Commit message: Updates data_aquisition.py to record data for the lstm

File: larcc_cell_description/urdf/larcc_cell.xacro (robot description, xacro)
@@ -18,5 +18,5 @@
     <xacro:include filename="$(find larcc_cell_description)/urdf/properties.xacro"/>
     <xacro:include filename="$(find ur_description)/urdf/inc/ur10e_macro.xacro"/>
-    <xacro:include filename="$(find realsense2_description)/urdf/test_d435i_camera.urdf.xacro" />
+<!--    <xacro:include filename="$(find realsense2_description)/urdf/test_d435i_camera.urdf.xacro" />-->
     <xacro:include filename="$(find gripper)/urdf/robotiq_arg2f_140_model_macro.xacro" />
     <xacro:include filename="$(find larcc_cell_description)/urdf/table.macro.xacro"/>
@@ -36,7 +36,7 @@
     </joint>
 <!--    Place d45i camera-->
-    <xacro:realsense2_camera parent="base_link" use_nominal_extrinsics="true">
-        <origin xyz="0.797 -0.803 0.432" rpy="3.135 2.462 -1.577"/>
-    </xacro:realsense2_camera>
+<!--    <xacro:realsense2_camera parent="base_link" use_nominal_extrinsics="true">-->
+<!--        <origin xyz="0.797 -0.803 0.432" rpy="3.135 2.462 -1.577"/>-->
+<!--    </xacro:realsense2_camera>-->
 <!--    Place gripper-->
     <xacro:robotiq_arg2f_140 prefix=""/>

Commit message: Solving launch problems: 1- Gripper and manipulator can be controlled simultaneously again 2- larcc xacro is correctly launched with ur10e external control available by MoveIt

File: larcc_cell_description/urdf/larcc_cell.xacro (robot description, xacro)
@@ -1,4 +1,4 @@
 <?xml version="1.0"?>
-<robot xmlns:xacro="http://wiki.ros.org/xacro" name="larcc_model">
+<robot xmlns:xacro="http://wiki.ros.org/xacro" name="larcc">
     <xacro:property name="M_PI" value="3.1415926535897931"/>
         <!-- Tables properties-->

File: ur_description/urdf/ur10e.xacro (robot description, xacro)
@@ -14,16 +14,35 @@
     Refer to 'inc/ur_macro.xacro' for more information.
   -->
-<!--  <link name="base_link"/>-->
-  <xacro:include filename="$(find ur_description)/urdf/inc/ur10e_macro.xacro"/>
-  <xacro:ur10e_robot prefix="" />
+    <link name="world"/>
+    <joint name="world_to_base_link" type="fixed">
+        <parent link="world"/>
+        <child link="base_link"/>
+        <origin xyz="0 0 -0.015" rpy="0 0 0"/>
+    </joint>
+    <joint name="world_to_robotiq_arg2f_base_link" type="fixed">
+        <parent link="world"/>
+        <child link="robotiq_arg2f_base_link"/>
+        <origin xyz="10 0 -0.5" rpy="0 0 0"/>
+    </joint>
+    <xacro:include filename="$(find ur_description)/urdf/inc/ur10e_macro.xacro"/>
+    <xacro:ur10e_robot prefix="" />
+    <xacro:include filename="$(find gripper)/urdf/robotiq_arg2f_140_model_macro.xacro" />
+<!--    Place gripper-->
+    <xacro:robotiq_arg2f_140 prefix=""/>
+<!--    <joint name="new_gripper_joint" type="fixed">-->
+<!--        <parent link="tool0"/>-->
+<!--        <child link="robotiq_arg2f_base_link"/>-->
+<!--        <origin xyz="0 0 0" rpy="0 0 1.5708"/>-->
+<!--&lt;!&ndash;    </joint>&ndash;&gt;-->
+<!--    </xacro:robotiq_arg2f_140>-->
 <!--  Sensor-->
-  <xacro:include filename="$(find realsense2_description)/urdf/test_d435i_camera.urdf.xacro" />
-  <xacro:realsense2_camera parent="base_link" use_nominal_extrinsics="true">
-<!--    For this manual calibration, drag the gripper (tool0_controller) to the camera mass
-        center and record here the tf values (/base_link to /tool0_controller).-->
-<!--    The second rotation value (P) you should add pi constant: 2.627 = −0,515 + pi -->
-<!--      <origin xyz="0.785 -0.839 0.426" rpy="-3.104 2.471 -1.613"/>-->
-      <origin xyz="0.797 -0.803 0.432" rpy="3.135 2.462 -1.577"/>
-  </xacro:realsense2_camera>
+<!--  <xacro:include filename="$(find realsense2_description)/urdf/test_d435i_camera.urdf.xacro" />-->
+<!--  <xacro:realsense2_camera parent="base_link" use_nominal_extrinsics="true">-->
+<!--&lt;!&ndash;    For this manual calibration, drag the gripper (tool0_controller) to the camera mass-->
+<!--        center and record here the tf values (/base_link to /tool0_controller).&ndash;&gt;-->
+<!--&lt;!&ndash;    The second rotation value (P) you should add pi constant: 2.627 = −0,515 + pi &ndash;&gt;-->
+<!--&lt;!&ndash;      <origin xyz="0.785 -0.839 0.426" rpy="-3.104 2.471 -1.613"/>&ndash;&gt;-->
+<!--      <origin xyz="0.797 -0.803 0.432" rpy="3.135 2.462 -1.577"/>-->
+<!--  </xacro:realsense2_camera>-->
 <!--  <xacro:realsense2_camera use_nominal_extrinsics="true">-->
 <!--  </xacro:realsense2_camera>-->
