Commit message: xacros, launches, urdfs, srdfs, update for remotely controling the robot with all the LARCC xacro (including tables, new FT sensor, gantry, gripper and manipulator).
This commit was used to create the new larcc_drivers repository (lardemua).

File: gripper/urdf/robotiq_arg2f_140_model_macro.xacro (robot description, xacro)
@@ -18,5 +18,5 @@
         <origin xyz="0 0 0" rpy="0 0 0" />
         <geometry>
-          <mesh filename="package://robotiq_2f_140_gripper_visualization/meshes/visual/robotiq_arg2f_${stroke}_outer_knuckle.stl" />
+          <mesh filename="package://gripper/meshes/visual/robotiq_arg2f_${stroke}_outer_knuckle.stl" />
         </geometry>
         <material name="">
@@ -27,5 +27,5 @@
         <origin xyz="0 0 0" rpy="0 0 0" />
         <geometry>
-          <mesh filename="package://robotiq_2f_140_gripper_visualization/meshes/collision/robotiq_arg2f_${stroke}_outer_knuckle.stl" />
+          <mesh filename="package://gripper/meshes/collision/robotiq_arg2f_${stroke}_outer_knuckle.stl" />
         </geometry>
       </collision>
@@ -48,5 +48,5 @@
         <origin xyz="0 0 0" rpy="0 0 0" />
         <geometry>
-          <mesh filename="package://robotiq_2f_140_gripper_visualization/meshes/visual/robotiq_arg2f_${stroke}_outer_finger.stl" />
+          <mesh filename="package://gripper/meshes/visual/robotiq_arg2f_${stroke}_outer_finger.stl" />
         </geometry>
         <material name="">
@@ -57,5 +57,5 @@
         <origin xyz="0 0 0" rpy="0 0 0" />
         <geometry>
-          <mesh filename="package://robotiq_2f_140_gripper_visualization/meshes/collision/robotiq_arg2f_${stroke}_outer_finger.stl" />
+          <mesh filename="package://gripper/meshes/collision/robotiq_arg2f_${stroke}_outer_finger.stl" />
         </geometry>
       </collision>
@@ -78,5 +78,5 @@
         <origin xyz="0 0 0" rpy="0 0 0" />
         <geometry>
-          <mesh filename="package://robotiq_2f_140_gripper_visualization/meshes/visual/robotiq_arg2f_${stroke}_inner_knuckle.stl" />
+          <mesh filename="package://gripper/meshes/visual/robotiq_arg2f_${stroke}_inner_knuckle.stl" />
         </geometry>
         <material name="">
@@ -87,5 +87,5 @@
         <origin xyz="0 0 0" rpy="0 0 0" />
         <geometry>
-          <mesh filename="package://robotiq_2f_140_gripper_visualization/meshes/collision/robotiq_arg2f_${stroke}_inner_knuckle.stl" />
+          <mesh filename="package://gripper/meshes/collision/robotiq_arg2f_${stroke}_inner_knuckle.stl" />
         </geometry>
       </collision>
@@ -108,5 +108,5 @@
         <origin xyz="0 0 0" rpy="0 0 0" />
         <geometry>
-          <mesh filename="package://robotiq_2f_140_gripper_visualization/meshes/visual/robotiq_arg2f_${stroke}_inner_finger.stl" />
+          <mesh filename="package://gripper/meshes/visual/robotiq_arg2f_${stroke}_inner_finger.stl" />
         </geometry>
         <material name="">
@@ -117,5 +117,5 @@
         <origin xyz="0 0 0" rpy="0 0 0" />
         <geometry>
-          <mesh filename="package://robotiq_2f_140_gripper_visualization/meshes/collision/robotiq_arg2f_${stroke}_inner_finger.stl" />
+          <mesh filename="package://gripper/meshes/collision/robotiq_arg2f_${stroke}_inner_finger.stl" />
         </geometry>
       </collision>

File: larcc_cell_description/urdf/larcc_cell.xacro (robot description, xacro)
@@ -39,10 +39,50 @@
 <!--        <origin xyz="0.797 -0.803 0.432" rpy="3.135 2.462 -1.577"/>-->
 <!--    </xacro:realsense2_camera>-->
+    <joint name="tool0-FT_sensor_base" type="fixed">
+        <parent link="tool0"/>
+        <child link="FT_sensor_base"/>
+        <origin xyz="0 0 0.003" rpy="0 0 1.5708"/>
+    </joint>
+    <link name="FT_sensor_base">
+        <visual>
+          <geometry>
+            <cylinder length="0.006" radius="0.05"/>
+          </geometry>
+          <material name="metalic_blue">
+            <color rgba="0.0118 0.5176 0.6706 1.0"/>
+          </material>
+        </visual>
+        <collision>
+          <geometry>
+            <cylinder length="0.006" radius="0.05"/>
+          </geometry>
+        </collision>
+    </link>
+    <joint name="FT_sensor_base-FT_sensor" type="fixed">
+        <parent link="FT_sensor_base"/>
+        <child link="FT_sensor"/>
+        <origin xyz="0 0 0.014" rpy="0 0 0"/>
+    </joint>
+    <link name="FT_sensor">
+        <visual>
+          <geometry>
+            <cylinder length="0.022" radius="0.04"/>
+          </geometry>
+          <material name="metalic_blue">
+            <color rgba="0.0118 0.5176 0.6706 1.0"/>
+          </material>
+        </visual>
+        <collision>
+          <geometry>
+            <cylinder length="0.022" radius="0.04"/>
+          </geometry>
+        </collision>
+    </link>
 <!--    Place gripper-->
     <xacro:robotiq_arg2f_140 prefix=""/>
-    <joint name="new_gripper_joint" type="fixed">
-        <parent link="tool0"/>
+    <joint name="gripper_joint" type="fixed">
+        <parent link="FT_sensor"/>
         <child link="robotiq_arg2f_base_link"/>
-        <origin xyz="0 0 0" rpy="0 0 1.5708"/>
+        <origin xyz="0 0 0.011" rpy="0 0 0"/>
     </joint>
 <!--    Place base table-->

File: ur_description/urdf/ur10e.xacro (robot description, xacro)
@@ -20,20 +20,19 @@
         <origin xyz="0 0 -0.015" rpy="0 0 0"/>
     </joint>
-    <joint name="world_to_robotiq_arg2f_base_link" type="fixed">
-        <parent link="world"/>
-        <child link="robotiq_arg2f_base_link"/>
-        <origin xyz="10 0 -0.5" rpy="0 0 0"/>
-    </joint>
+<!--    <joint name="world_to_robotiq_arg2f_base_link" type="fixed">-->
+<!--        <parent link="world"/>-->
+<!--        <child link="robotiq_arg2f_base_link"/>-->
+<!--        <origin xyz="10 0 -0.5" rpy="0 0 0"/>-->
+<!--    </joint>-->
     <xacro:include filename="$(find ur_description)/urdf/inc/ur10e_macro.xacro"/>
     <xacro:ur10e_robot prefix="" />
+    <joint name="gripper_joint" type="fixed">
+        <parent link="tool0"/>
+        <child link="robotiq_arg2f_base_link"/>
+        <origin xyz="0 0 0" rpy="0 0 1.5708"/>
+    </joint>
+<!--    Place gripper-->
     <xacro:include filename="$(find gripper)/urdf/robotiq_arg2f_140_model_macro.xacro" />
-<!--    Place gripper-->
     <xacro:robotiq_arg2f_140 prefix=""/>
-<!--    <joint name="new_gripper_joint" type="fixed">-->
-<!--        <parent link="tool0"/>-->
-<!--        <child link="robotiq_arg2f_base_link"/>-->
-<!--        <origin xyz="0 0 0" rpy="0 0 1.5708"/>-->
-<!--&lt;!&ndash;    </joint>&ndash;&gt;-->
-<!--    </xacro:robotiq_arg2f_140>-->
 <!--  Sensor-->
 <!--  <xacro:include filename="$(find realsense2_description)/urdf/test_d435i_camera.urdf.xacro" />-->
@@ -47,11 +46,3 @@
 <!--  <xacro:realsense2_camera use_nominal_extrinsics="true">-->
 <!--  </xacro:realsense2_camera>-->
-  <!-- Gripper -->
-<!--  <xacro:include filename="$(find robotiq_2f_140_gripper_visualization)/urdf/robotiq_arg2f_140.xacro" />-->
-<!--  <xacro:robotiq_arg2f_140_model parent="base_link">-->
-<!--      <origin xyz="1.7 -0.833 0.424 " rpy="3.073 2.627 -1.650"/>-->
-<!--  </xacro:robotiq_arg2f_140_model>-->
-<!--&lt;!&ndash;   Gripper &ndash;&gt;-->
-<!--  <xacro:include filename="$(find robotiq_2f_140_gripper_visualization)/urdf/robotiq_arg2f_140.xacro" />-->
-<!--  <xacro:robotiq_arg2f_140_model/>-->
 </robot>
